File: Brewnode_MCU_Adapter.kicad_pcb (KiCad board)
At the start: 2 copper layers, 0 parts

Commit message: PCB Sent to production
Parts:
- added J17: 16p FPC, Tobbe_Hirose:Hirose_FH34_FPC_16, F.Cu at (119.9, 97.8)
- added REF**: MountingHole_4mm, MountingHole:MountingHole_4mm, F.Cu at (181.1, 110.5)
- added REF**: MountingHole_4mm, MountingHole:MountingHole_4mm, F.Cu at (120.9, 110.5)
- added REF**: MountingHole_4mm, MountingHole:MountingHole_4mm, F.Cu at (120.9, 85.1)
- added REF**: MountingHole_4mm, MountingHole:MountingHole_4mm, F.Cu at (181.1, 85.1)
- added U1: ESP32_DevKit_V1_DOIT, ESP32_DevKit_V1_DOIT:esp32_devkit_v1_doit, F.Cu at (131.3, 97.8)
Routing:
- net +5V: track 0.00 -> 67.0 mm, vias 0 -> 1
- net /3V3_IOEXP_INT: track 0.00 -> 57.5 mm, vias 0 -> 2
- net +3V3: track 0.00 -> 57.1 mm
- net /PORT1: track 0.00 -> 42.4 mm, vias 0 -> 2
- net /PORT2: track 0.00 -> 39.9 mm, vias 0 -> 2
- net /PORT3: track 0.00 -> 35.2 mm, vias 0 -> 2
- net /PORT4: track 0.00 -> 33.1 mm, vias 0 -> 2
- net /3V3_SCL: track 0.00 -> 31.4 mm, vias 0 -> 2
- net /3V3_SDA: track 0.00 -> 30.7 mm, vias 0 -> 2
- net /3V3_ADC_INT: track 0.00 -> 20.3 mm, vias 0 -> 2
- net GND: track 0.00 -> 9.97 mm, vias 0 -> 2
- added copper zone on B.Cu, net GND
Other:
- board outline added: 72.1 x 36.1 mm
- net class Default: clearance 0.1524 -> 0.2; trace_width 0.1524 -> 0.25; via_dia 0.6 -> 0.8; via_drill 0.3 -> 0.4
- rule pad_to_mask_clearance: 0.0508 -> 0
- rule trace_clearance: 0.1524 -> 0.2
- rule trace_min: 0.1524 -> 0.2
- rule via_min_size: 0.6 -> 0.4
- board text added: "Brewnode V1 Adapter"
- board text added: "ESP32 Devkit V1 DOIT"
