File: Brewnode_MCU_Adapter.kicad_pcb (KiCad board)
At the start: 2 copper layers, 72.1 x 36.1 mm, 6 parts, among them J17 16p FPC, U1 ESP32_DevKit_V1_DOIT

Commit message: PCB Produced
Parts:
- J17: moved to B.Cu
- turned J17 to 90 degrees
Routing:
- net GND: track 9.97 -> 27.7 mm, vias 2 -> 3
- net /3V3_IOEXP_INT: track 57.5 -> 44.7 mm, vias 2 -> 1
- net +5V: track 67.0 -> 57.8 mm, vias 1 -> 0
- net /3V3_SCL: track 31.4 -> 23.4 mm, vias 2 -> 1
- net /3V3_ADC_INT: track 20.3 -> 22.3 mm, vias 2 -> 1
- net /PORT4: track 33.1 -> 31.6 mm, vias 2 -> 1
- net +3V3: track 57.1 -> 55.8 mm, vias 0 -> 1
- net /PORT1: track 42.4 -> 43.3 mm, vias 2 -> 1
- net /3V3_SDA: track 30.7 -> 30.1 mm, vias 2 -> 1
- net /PORT3: track 35.2 -> 34.9 mm, vias 2 -> 1
- net /PORT2: track 39.9 -> 40.1 mm, vias 2 -> 1
