File: Brewnode_MCU_Adapter.sch (KiCad schematic (older format))
At the start: 0 parts

Commit message: PCB Sent to production
Parts:
- added J17: 16p FPC, Tobbe_Hirose:Hirose_FH34_FPC_16, symbol Connector_Generic:Conn_01x16
- added U1: ESP32_DevKit_V1_DOIT, ESP32_DevKit_V1_DOIT:esp32_devkit_v1_doit, symbol ESP32_DevKit_V1_DOIT:ESP32_DevKit_V1_DOIT
Connections:
- net labels added: +3V3, +5V, 3V3_ADC_INT, 3V3_IOEXP_INT, 3V3_SCL, 3V3_SDA, GND, PORT1, PORT2, PORT3, PORT4
- wire segments 0 -> 62
- no-connect marks 0 -> 1
